Commit message: added gitignore

File: src/my_gamefield/description/robot.urdf.xacro (robot description, xacro)
@@ -1,366 +1,5 @@
 <?xml version="1.0"?>
-<robot name="game_field">
-  <!-- Root Frame -->
-  <link name="map"/>
-  <!-- Static Joint from map to field_base -->
-  <joint name="map_to_field_base" type="fixed">
-    <parent link="map"/>
-    <child link="field_base"/>
-    <origin xyz="0 0 0" rpy="0 0 0"/> <!-- Adjust if necessary -->
-  </joint>
-  <!-- Main Field Base -->
-  <link name="field_base">
-    <visual>
-      <geometry>
-        <box size="15.0 8.0 0.01"/> <!-- Main field dimensions -->
-      </geometry>
-      <material name="field_surface">
-        <color rgba="1.0 1.0 1.0 0.5"/> <!-- Semi-transparent white -->
-      </material>
-    </visual>
-    <collision>
-      <geometry>
-        <box size="15.0 8.0 0.01"/>
-      </geometry>
-    </collision>
-    <!-- Inertial properties -->
-    <inertial>
-      <mass value="1.0"/>
-      <origin xyz="0 0 0" rpy="0 0 0"/>
-      <inertia ixx="1.0" ixy="0.0" ixz="0.0" iyy="1.0" iyz="0.0" izz="1.0"/>
-    </inertial>
-  </link>
-  <!-- Left Hoop -->
-  <link name="hoop_left">
-    <visual>
-      <geometry>
-        <cylinder radius="0.225" length="3.05"/> <!-- Hoop post dimensions -->
-      </geometry>
-      <material name="hoop_material">
-        <color rgba="0.8 0.3 0.3 1.0"/> <!-- Red hoop -->
-      </material>
-    </visual>
-    <collision>
-      <geometry>
-        <cylinder radius="0.225" length="3.05"/>
-      </geometry>
-    </collision>
-    <!-- Inertial properties -->
-    <inertial>
-      <mass value="1.0"/>
-      <origin xyz="0 0 0" rpy="0 0 0"/>
-      <inertia ixx="0.1" ixy="0.0" ixz="0.0" iyy="0.1" iyz="0.0" izz="0.1"/>
-    </inertial>
-  </link>
-  <joint name="hoop_left_joint" type="fixed">
-    <parent link="field_base"/>
-    <child link="hoop_left"/>
-    <origin xyz="7.2 0.0 1.525"/> <!-- Position of the left hoop -->
-  </joint>
-  <!-- Right Hoop -->
-  <link name="hoop_right">
-    <visual>
-      <geometry>
-        <cylinder radius="0.225" length="3.05"/> <!-- Hoop post dimensions -->
-      </geometry>
-      <material name="hoop_material">
-        <color rgba="0.8 0.3 0.3 1.0"/> <!-- Red hoop -->
-      </material>
-    </visual>
-    <collision>
-      <geometry>
-        <cylinder radius="0.225" length="3.05"/>
-      </geometry>
-    </collision>
-    <!-- Inertial properties -->
-    <inertial>
-      <mass value="1.0"/>
-      <origin xyz="0 0 0" rpy="0 0 0"/>
-      <inertia ixx="0.1" ixy="0.0" ixz="0.0" iyy="0.1" iyz="0.0" izz="0.1"/>
-    </inertial>
-  </link>
-  <joint name="hoop_right_joint" type="fixed">
-    <parent link="field_base"/>
-    <child link="hoop_right"/>
-    <origin xyz="-7.2 -0.0 1.525"/> <!-- Position of the right hoop -->
-  </joint>
-  <!-- Key Zone Left -->
-  <link name="key_zone_left">
-    <visual>
-      <geometry>
-        <box size="2.5 1.8 0.01"/> <!-- Key zone dimensions -->
-      </geometry>
-      <material name="zone_material">
-        <color rgba="0.5 0.5 0.5 1.0"/> <!-- Grey color for the field -->
-      </material>
-    </visual>
-    <collision>
-      <geometry>
-        <box size="2.5 1.8 0.01"/>
-      </geometry>
-    </collision>
-    <!-- Inertial properties -->
-    <inertial>
-      <mass value="0.5"/>
-      <origin xyz="0 0 0" rpy="0 0 0"/>
-      <inertia ixx="0.1" ixy="0.0" ixz="0.0" iyy="0.1" iyz="0.0" izz="0.1"/>
-    </inertial>
-  </link>
-  <joint name="key_zone_left_joint" type="fixed">
-    <parent link="field_base"/>
-    <child link="key_zone_left"/>
-    <origin xyz="6.25 0.0 0.005"/> <!-- Position in front of the left hoop -->
-  </joint>
-  <!-- Key Zone Right -->
-  <link name="key_zone_right">
-    <visual>
-      <geometry>
-        <box size="2.5 1.8 0.01"/> <!-- Key zone dimensions -->
-      </geometry>
-      <material name="zone_material">
-        <color rgba="0.5 0.5 0.5 1.0"/> <!-- Grey color for the field -->
-      </material>
-    </visual>
-    <collision>
-      <geometry>
-        <box size="2.5 1.8 0.01"/>
-      </geometry>
-    </collision>
-    <!-- Inertial properties -->
-    <inertial>
-      <mass value="0.5"/>
-      <origin xyz="0 0 0" rpy="0 0 0"/>
-      <inertia ixx="0.1" ixy="0.0" ixz="0.0" iyy="0.1" iyz="0.0" izz="0.1"/>
-    </inertial>
-  </link>
-  <joint name="key_zone_right_joint" type="fixed">
-    <parent link="field_base"/>
-    <child link="key_zone_right"/>
-    <origin xyz="-6.25 0.0 0.005"/> <!-- Position in front of the right hoop -->
-  </joint>
-  <!-- Center Line -->
-  <link name="center_line">
-    <visual>
-      <geometry>
-        <box size="0.05 8.0 0.01"/> <!-- Center line dimensions -->
-      </geometry>
-      <material name="line_material">
-        <color rgba="1.0 1.0 1.0 1.0"/> <!-- White line -->
-      </material>
-    </visual>
-    <collision>
-      <geometry>
-        <box size="0.05 8.0 0.01"/>
-      </geometry>
-    </collision>
-    <!-- Inertial properties -->
-    <inertial>
-      <mass value="0.1"/>
-      <origin xyz="0 0 0" rpy="0 0 0"/>
-      <inertia ixx="0.1" ixy="0.0" ixz="0.0" iyy="0.1" iyz="0.0" izz="0.1"/>
-    </inertial>
-  </link>
-  <joint name="center_line_joint" type="fixed">
-    <parent link="field_base"/>
-    <child link="center_line"/>
-    <origin xyz="0.0 0.0 0.005"/> <!-- Positioned at the center of the field -->
-  </joint>
-  <!-- Goal Area Rectangle (Left) -->
-  <link name="left_goal_area">
-	<visual>
-  	<geometry>
-    	<box size="2.5 1.8 0.01"/> <!-- Size: 4500mm x 1800mm -->
-  	</geometry>
-  	<material name="white">
-    	<color rgba="1.0 1.0 1.0 1.0"/> <!-- White zone -->
-  	</material>
-	</visual>
-	<collision>
-  	<geometry>
-    	<box size="2.5 1.8 0.01"/>
-  	</geometry>
-	</collision>
-  </link>
-  <joint name="left_goal_joint" type="fixed">
-	<parent link="field_base"/>
-	<child link="left_goal_area"/>
-	<origin xyz="-6.25 0 0.01" rpy="0 0 0"/> <!-- Position relative to field -->
-  </joint>
- <!-- Goal Area Rectangle (Right) -->
-  <link name="right_goal_area">
-	<visual>
-  	<geometry>
-    	<box size="2.5 1.8 0.01"/> <!-- Size: 4500mm x 1800mm -->
-  	</geometry>
-  	<material name="white">
-    	<color rgba="1.0 1.0 1.0 1.0"/> <!-- White zone -->
-  	</material>
-	</visual>
-	<collision>
-  	<geometry>
-    	<box size="2.5 1.8 0.01"/>
-  	</geometry>
-	</collision>
-  </link>
-  <joint name="right_goal_joint" type="fixed">
-	<parent link="field_base"/>
-	<child link="right_goal_area"/>
-	<origin xyz="6.25 0 0.01" rpy="0 0 0"/> <!-- Position relative to field -->
-  </joint>
- <!-- Fence_right-->
-  <link name="fence_right">
-	<visual>
-  	<geometry>
-    	<box size="15.1 0.05 0.05"/> <!-- Length: 15m, Thickness: 0.1m, Height: 2m -->
-  	</geometry>
-  	<material name="gray">
-        <color rgba="0.8 0.3 0.3 1.0"/> <!-- Red -->
-  	</material>
-	</visual>
-	<collision>
-  	<geometry>
-    	<box size="15.1 0.05 0.05"/>
-  	</geometry>
-	</collision>
-	<inertial>
-  	<mass value="5.0"/>
-  	<origin xyz="0 0 0" rpy="0 0 0"/>
-  	<inertia ixx="1.0" ixy="0.0" ixz="0.0" iyy="1.0" iyz="0.0" izz="1.0"/>
-	</inertial>
-  </link>
-  <joint name="fence_joint_right" type="fixed">
-	<parent link="field_base"/>
-	<child link="fence_right"/>
-	<origin xyz="0.0 -4.0 0.0" rpy="0 0 0"/> <!-- Positioned behind the field -->
-  </joint>
- <!-- Fence_left -->
-  <link name="fence_left">
-	<visual>
-  	<geometry>
-    	<box size="15.1 0.05 0.05"/> <!-- Length: 15m, Thickness: 0.1m, Height: 2m -->
-  	</geometry>
-  	<material name="gray">
-        <color rgba="0.8 0.3 0.3 1.0"/> <!-- Red -->
-  	</material>
-	</visual>
-	<collision>
-  	<geometry>
-    	<box size="15.1 0.05 0.05"/>
-  	</geometry>
-	</collision>
-	<inertial>
-  	<mass value="5.0"/>
-  	<origin xyz="0 0 0" rpy="0 0 0"/>
-  	<inertia ixx="1.0" ixy="0.0" ixz="0.0" iyy="1.0" iyz="0.0" izz="1.0"/>
-	</inertial>
-  </link>
-  <joint name="fence_joint_left" type="fixed">
-	<parent link="field_base"/>
-	<child link="fence_left"/>
-	<origin xyz="0.0 4.0 0.0" rpy="0 0 0"/> <!-- Positioned behind the field -->
-  </joint>
-<!-- Fence_left -->
-  <link name="fence_north">
-	<visual>
-  	<geometry>
-    	<box size="0.05 8.0 0.05"/> <!-- Length: 15m, Thickness: 0.1m, Height: 2m -->
-  	</geometry>
-  	<material name="gray">
-        <color rgba="0.8 0.3 0.3 1.0"/> <!-- Red -->
-  	</material>
-	</visual>
-	<collision>
-  	<geometry>
-    	<box size="0.05 8.0 0.05"/>
-  	</geometry>
-	</collision>
-	<inertial>
-  	<mass value="5.0"/>
-  	<origin xyz="0 0 0" rpy="0 0 0"/>
-  	<inertia ixx="1.0" ixy="0.0" ixz="0.0" iyy="1.0" iyz="0.0" izz="1.0"/>
-	</inertial>
-  </link>
-  <joint name="fence_joint_north" type="fixed">
-	<parent link="field_base"/>
-	<child link="fence_north"/>
-	<origin xyz="7.55 0.0 0.0" rpy="0 0 0"/> <!-- Positioned behind the field -->
-  </joint>
-<!-- Fence_left -->
-  <link name="fence_west">
-	<visual>
-  	<geometry>
-    	<box size="0.05 8.0 0.05"/> <!-- Length: 15m, Thickness: 0.1m, Height: 2m -->
-  	</geometry>
-  	<material name="gray">
-        <color rgba="0.8 0.3 0.3 1.0"/> <!-- Red -->
-  	</material>
-	</visual>
-	<collision>
-  	<geometry>
-    	<box size="0.05 8.0 0.05"/>
-  	</geometry>
-	</collision>
-	<inertial>
-  	<mass value="5.0"/>
-  	<origin xyz="0 0 0" rpy="0 0 0"/>
-  	<inertia ixx="1.0" ixy="0.0" ixz="0.0" iyy="1.0" iyz="0.0" izz="1.0"/>
-	</inertial>
-  </link>
-  <joint name="fence_joint_west" type="fixed">
-	<parent link="field_base"/>
-	<child link="fence_west"/>
-	<origin xyz="-7.55 0.0 0.0" rpy="0 0 0"/> <!-- Positioned behind the field -->
-  </joint>
- <!-- 3-Point Line (Left) -->
-  <link name="left_three_point_line">
-	<visual>
-  	<geometry>
-    	<cylinder radius="3.1" length="0.0"/> <!-- Line thickness: 50mm, Arc length -->
-  	</geometry>
-  	<material name="white">
-    	<color rgba="1.0 1.0 1.0 1.0"/> <!-- White color -->
-  	</material>
-	</visual>
-	<collision>
-  	<geometry>
-    	<cylinder radius="3.1" length="0.0"/>
-  	</geometry>
-	</collision>
-	<inertial>
-  	<mass value="0.1"/>
-  	<origin xyz="0 0 0" rpy="0 0 0"/>
-  	<inertia ixx="0.001" ixy="0.0" ixz="0.0" iyy="0.001" iyz="0.0" izz="0.001"/>
-	</inertial>
-  </link>
-  <joint name="left_three_point_line_joint" type="fixed">
-	<parent link="field_base"/>
-	<child link="left_three_point_line"/>
-	<origin xyz="-6.75 0.0 0.01" rpy="0 0 0"/> <!-- Positioned for the left arc -->
-  </joint>
-<!-- 3-Point Line (right) -->
-  <link name="right_three_point_line">
-	<visual>
-  	<geometry>
-    	<cylinder radius="3.1" length="0.0"/> <!-- Line thickness: 50mm, Arc length -->
-  	</geometry>
-  	<material name="green">
-    	<color rgba="0 0 0 0"/> <!-- White color -->
-  	</material>
-	</visual>
-	<collision>
-  	<geometry>
-    	<cylinder radius="3.1" length="0.0"/>
-  	</geometry>
-	</collision>
-	<inertial>
-  	<mass value="0.1"/>
-  	<origin xyz="0 0 0" rpy="0 0 0"/>
-  	<inertia ixx="0.001" ixy="0.0" ixz="0.0" iyy="0.001" iyz="0.0" izz="0.001"/>
-	</inertial>
-  </link>
-  <joint name="right_three_point_line_joint" type="fixed">
-	<parent link="field_base"/>
-	<child link="right_three_point_line"/>
-	<origin xyz="6.75 0.0 0.01" rpy="0 0 0"/> <!-- Positioned for the left arc -->
-  </joint>
+<robot xmlns:xacro="http://www.ros.org/wiki/xacro"  name="game_field">
+		<xacro:include filename="gamefield.xacro"/>
+		<xacro:include filename="robot_model.xacro"/>
 </robot>

File: src/my_gamefield/description/robot_model.xacro (robot description, xacro)
@@ -5,5 +5,5 @@
 <xacro:if value="${team == 'red'}">
 <joint name = "map_joint" type = "fixed">
-<parent link = "field_base_link"/>
+<parent link = "field_base"/>
 <child link = "map"/>
 <origin xyz = "-8.5780 0 0" rpy = "0 0 -1.57075"/>
@@ -12,5 +12,5 @@
 <xacro:if value="${team == 'blue'}">
 <joint name = "map_joint" type = "fixed">
-<parent link = "field_base_link"/>
+<parent link = "field_base"/>
 <child link = "map"/>
 <origin xyz = "0 0 0" rpy = "0 0 -1.57075"/>
@@ -22,33 +22,3 @@
 </visual>
 </link>
-<!--
-<joint name = "chasis_joint" type = "fixed">
-<parent link = "base_link"/>
-<child link = "chasis_link"/>
-<origin xyz = "0 0 0"/>
-</joint>
-<link name = "chasis_link">
-<visual>
-<origin xyz = "0 0 0.135"/>
-<geometry>
-<box size = "0.25 0.25 0.25"/>
-</geometry>
-<material name = "pink"/>
-</visual>
-</link>
-<joint name = "camera_joint" type = "fixed">
-<parent link = "chasis_link"/>
-<child link = "camera_link"/>
-<origin xyz = "0 0 0"/>
-</joint>
-<link name = "camera_link">
-<visual>
-<material name = "grey"/>
-<origin xyz = "-0.125 0 0.30"/>
-<geometry>
-<box size = "0.10 0.1 0.10"/>
-</geometry>
-</visual>
-</link>
--->
 </robot>
